File: My MCU datalogger.kicad_sch (KiCad schematic)
At the start: 6 parts

Commit message: build in progress
Parts:
- added R2, R3, R4, R5, R6, R7: R, symbol Device:R
- renumbered C25 to C5
Changed lines of the file:
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@@
     (effects (font (size 5 5) (thickness 1)) (justify left bottom))
   )
+  (symbol (lib_id "Device:R") (at 144.78 77.47 0) (unit 1)
+    (in_bom yes) (on_board yes) (fields_autoplaced)
+    (property "Reference" "R7" (id 0) (at 147.32 76.1999 0)
+      (effects (font (size 1.27 1.27)) (justify left))
+    )
+    (property "Value" "R" (id 1) (at 147.32 78.7399 0)
+      (effects (font (size 1.27 1.27)) (justify left))
+    )
+    (property "Footprint" "" (id 2) (at 143.002 77.47 90)
+      (effects (font (size 1.27 1.27)) hide)
+    )
+    (property "Datasheet" "~" (id 3) (at 144.78 77.47 0)
+      (effects (font (size 1.27 1.27)) hide)
+    )
+    (pin "1")
+    (pin "2")
+  )
   (symbol (lib_id "Device:C") (at 160.02 55.88 0) (unit 1)
     (in_bom yes) (on_board yes) (fields_autoplaced)
@@
     (pin "2")
   )
+  (symbol (lib_id "Device:R") (at 104.14 77.47 0) (unit 1)
+    (in_bom yes) (on_board yes) (fields_autoplaced)
+    (property "Reference" "R3" (id 0) (at 106.68 76.1999 0)
+      (effects (font (size 1.27 1.27)) (justify left))
+    )
+    (property "Value" "R" (id 1) (at 106.68 78.7399 0)
+      (effects (font (size 1.27 1.27)) (justify left))
+    )
+    (property "Footprint" "" (id 2) (at 102.362 77.47 90)
+      (effects (font (size 1.27 1.27)) hide)
+    )
+    (property "Datasheet" "~" (id 3) (at 104.14 77.47 0)
+      (effects (font (size 1.27 1.27)) hide)
+    )
+    (pin "1")
+    (pin "2")
+  )
   (symbol (lib_id "Device:C") (at 172.72 55.88 0) (unit 1)
     (in_bom yes) (on_board yes) (fields_autoplaced)
-    (property "Reference" "C25" (id 0) (at 176.53 54.6099 0)
+    (property "Reference" "C5" (id 0) (at 176.53 54.6099 0)
       (effects (font (size 1.27 1.27)) (justify left))
     )
@@
     (pin "2")
   )
+  (symbol (lib_id "Device:R") (at 135.89 77.47 0) (unit 1)
+    (in_bom yes) (on_board yes) (fields_autoplaced)
+    (property "Reference" "R6" (id 0) (at 138.43 76.1999 0)
+      (effects (font (size 1.27 1.27)) (justify left))
+    )
+    (property "Value" "R" (id 1) (at 138.43 78.7399 0)
+      (effects (font (size 1.27 1.27)) (justify left))
+    )
+    (property "Footprint" "" (id 2) (at 134.112 77.47 90)
+      (effects (font (size 1.27 1.27)) hide)
+    )
+    (property "Datasheet" "~" (id 3) (at 135.89 77.47 0)
+      (effects (font (size 1.27 1.27)) hide)
+    )
+    (pin "1")
+    (pin "2")
+  )
   (symbol (lib_id "Device:C") (at 132.08 55.88 0) (unit 1)
     (in_bom yes) (on_board yes) (fields_autoplaced)
@@
     )
     (property "Datasheet" "~" (id 3) (at 132.08 55.88 0)
+      (effects (font (size 1.27 1.27)) hide)
+    )
+    (pin "1")
+    (pin "2")
+  )
+  (symbol (lib_id "Device:R") (at 93.98 77.47 0) (unit 1)
+    (in_bom yes) (on_board yes) (fields_autoplaced)
+    (property "Reference" "R2" (id 0) (at 96.52 76.1999 0)
+      (effects (font (size 1.27 1.27)) (justify left))
+    )
+    (property "Value" "R" (id 1) (at 96.52 78.7399 0)
+      (effects (font (size 1.27 1.27)) (justify left))
+    )
+    (property "Footprint" "" (id 2) (at 92.202 77.47 90)
+      (effects (font (size 1.27 1.27)) hide)
+    )
+    (property "Datasheet" "~" (id 3) (at 93.98 77.47 0)
+      (effects (font (size 1.27 1.27)) hide)
+    )
+    (pin "1")
+    (pin "2")
+  )
+  (symbol (lib_id "Device:R") (at 125.73 77.47 0) (unit 1)
+    (in_bom yes) (on_board yes) (fields_autoplaced)
+    (property "Reference" "R5" (id 0) (at 128.27 76.1999 0)
+      (effects (font (size 1.27 1.27)) (justify left))
+    )
+    (property "Value" "R" (id 1) (at 128.27 78.7399 0)
+      (effects (font (size 1.27 1.27)) (justify left))
+    )
+    (property "Footprint" "" (id 2) (at 123.952 77.47 90)
+      (effects (font (size 1.27 1.27)) hide)
+    )
+    (property "Datasheet" "~" (id 3) (at 125.73 77.47 0)
+      (effects (font (size 1.27 1.27)) hide)
+    )
+    (pin "1")
+    (pin "2")
+  )
+  (symbol (lib_id "Device:R") (at 116.84 77.47 0) (unit 1)
+    (in_bom yes) (on_board yes) (fields_autoplaced)
+    (property "Reference" "R4" (id 0) (at 119.38 76.1999 0)
+      (effects (font (size 1.27 1.27)) (justify left))
+    )
+    (property "Value" "R" (id 1) (at 119.38 78.7399 0)
+      (effects (font (size 1.27 1.27)) (justify left))
+    )
+    (property "Footprint" "" (id 2) (at 115.062 77.47 90)
+      (effects (font (size 1.27 1.27)) hide)
+    )
+    (property "Datasheet" "~" (id 3) (at 116.84 77.47 0)
       (effects (font (size 1.27 1.27)) hide)
     )
@@
     )
     (path "/5cfaff8f-4cb1-4092-acac-68ea8803d576"
-      (reference "C25") (unit 1) (value "C") (footprint "")
+      (reference "C5") (unit 1) (value "C") (footprint "")
     )
     (path "/c63b5fc8-661c-44e7-ac4b-00c9fb9e97ae"
       (reference "R1") (unit 1) (value "R") (footprint "")
     )
-  )
+    (path "/7e80ce5c-a2c9-412f-a84c-0638b490e970"
+      (reference "R2") (unit 1) (value "R") (footprint "")
+    )
+    (path "/53802d6b-42d5-42e1-af71-9bc8cee694a1"
+      (reference "R3") (unit 1) (value "R") (footprint "")
+    )
+    (path "/9dd523ff-b43a-43b7-a9af-c2ccfacb1997"
+      (reference "R4") (unit 1) (value "R") (footprint "")
+    )
+    (path "/87a3a773-fe73-42f4-9d3a-a7a67ac8acce"
+      (reference "R5") (unit 1) (value "R") (footprint "")
+    )
+    (path "/65028966-0ecc-41eb-92ed-c1bdfd67235f"
+      (reference "R6") (unit 1) (value "R") (footprint "")
+    )
+    (path "/01d22717-f17f-4a5c-b3aa-b3625d2b6850"
+      (reference "R7") (unit 1) (value "R") (footprint "")
+    )
+  )

Commit message: build in progress
Parts:
- added BT1: Battery, symbol Device:Battery
- added D1, D2: LED, symbol Device:LED
- added H1, H2, H3, H4: MountingHole, symbol Mechanical:MountingHole
- added J1, J3: Conn_01x04_Male, symbol Connector:Conn_01x04_Male
- added J2: Conn_01x09_Male, symbol Connector:Conn_01x09_Male
- added J4: Conn_02x03_Odd_Even, symbol Connector_Generic:Conn_02x03_Odd_Even
- added U1: 24LC1025, symbol Memory_EEPROM:24LC1025
- added U2: 24LC1025, Package_SO:SOIC-8_3.9x4.9mm_P1.27mm, symbol Memory_EEPROM:24LC1025
- added U?: ATMEGA328P-AU, digikey-footprints:TQFP-32_7x7mm, symbol dk_Embedded-Microcontrollers:ATMEGA328P-AU
- added Y1, Y2: Crystal, symbol Device:Crystal
- C1: value C -> 0,1uF
- C2, C3: value C -> 22pF
- C4: value C -> 0.1uF
- C5: value C -> 100nF
- R1, R2, R6: value R -> 10K
- R3, R4: value R -> 4.7K
- R5, R7: value R -> 330
Other:
- note removed: "MCU Data logger © 2022 by PC Soft War"
- company: PC Software -> PC Soft War

Commit message: build in progress
Parts:
- added U2: DS1307Z, SO08-TIGHT, symbol SparkFun-Clocks:DS1307Z
- gave numbers to parts that had none: 1
- renumbered U2 to U3
Other:
- moved on the sheet: U1, U3
Changed lines of the file:
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@@
     )
   )
-  (symbol (lib_id "Memory_EEPROM:24LC1025") (at 137.16 97.79 0) (unit 1)
-    (in_bom yes) (on_board yes) (fields_autoplaced)
-    (property "Reference" "U1" (id 0) (at 139.1794 87.63 0)
-      (effects (font (size 1.27 1.27)) (justify left))
-    )
-    (property "Value" "24LC1025" (id 1) (at 139.1794 90.17 0)
-      (effects (font (size 1.27 1.27)) (justify left))
-    )
-    (property "Footprint" "" (id 2) (at 137.16 97.79 0)
-      (effects (font (size 1.27 1.27)) hide)
-    )
-    (property "Datasheet" "http://ww1.microchip.com/downloads/en/DeviceDoc/21941B.pdf" (id 3) (at 137.16 97.79 0)
+  (symbol (lib_id "Memory_EEPROM:24LC1025") (at 127 111.76 0) (unit 1)
+    (in_bom yes) (on_board yes) (fields_autoplaced)
+    (property "Reference" "U1" (id 0) (at 129.0194 101.6 0)
+      (effects (font (size 1.27 1.27)) (justify left))
+    )
+    (property "Value" "24LC1025" (id 1) (at 129.0194 104.14 0)
+      (effects (font (size 1.27 1.27)) (justify left))
+    )
+    (property "Footprint" "" (id 2) (at 127 111.76 0)
+      (effects (font (size 1.27 1.27)) hide)
+    )
+    (property "Datasheet" "http://ww1.microchip.com/downloads/en/DeviceDoc/21941B.pdf" (id 3) (at 127 111.76 0)
       (effects (font (size 1.27 1.27)) hide)
     )
@@
     (pin "2")
   )
-  (symbol (lib_id "Memory_EEPROM:24LC1025") (at 166.37 97.79 0) (unit 1)
-    (in_bom yes) (on_board yes) (fields_autoplaced)
-    (property "Reference" "U2" (id 0) (at 168.3894 87.63 0)
-      (effects (font (size 1.27 1.27)) (justify left))
-    )
-    (property "Value" "24LC1025" (id 1) (at 168.3894 90.17 0)
-      (effects (font (size 1.27 1.27)) (justify left))
-    )
-    (property "Footprint" "Package_SO:SOIC-8_3.9x4.9mm_P1.27mm" (id 2) (at 166.37 97.79 0)
-      (effects (font (size 1.27 1.27)) hide)
-    )
-    (property "Datasheet" "http://ww1.microchip.com/downloads/en/DeviceDoc/21941B.pdf" (id 3) (at 166.37 97.79 0)
+  (symbol (lib_id "Memory_EEPROM:24LC1025") (at 184.15 110.49 0) (unit 1)
+    (in_bom yes) (on_board yes) (fields_autoplaced)
+    (property "Reference" "U3" (id 0) (at 186.1694 100.33 0)
+      (effects (font (size 1.27 1.27)) (justify left))
+    )
+    (property "Value" "24LC1025" (id 1) (at 186.1694 102.87 0)
+      (effects (font (size 1.27 1.27)) (justify left))
+    )
+    (property "Footprint" "Package_SO:SOIC-8_3.9x4.9mm_P1.27mm" (id 2) (at 184.15 110.49 0)
+      (effects (font (size 1.27 1.27)) hide)
+    )
+    (property "Datasheet" "http://ww1.microchip.com/downloads/en/DeviceDoc/21941B.pdf" (id 3) (at 184.15 110.49 0)
       (effects (font (size 1.27 1.27)) hide)
     )
@@
     (pin "2")
   )
+  (symbol (lib_id "SparkFun-Clocks:DS1307Z") (at 154.94 110.49 0) (unit 1)
+    (in_bom yes) (on_board yes) (fields_autoplaced)
+    (property "Reference" "U2" (id 0) (at 156.21 97.79 0)
+      (effects (font (size 1.143 1.143)))
+    )
+    (property "Value" "DS1307Z" (id 1) (at 156.21 100.33 0)
+      (effects (font (size 1.143 1.143)))
+    )
+    (property "Footprint" "SO08-TIGHT" (id 2) (at 154.94 101.6 0)
+      (effects (font (size 0.508 0.508)) hide)
+    )
+    (property "Datasheet" "" (id 3) (at 154.94 110.49 0)
+      (effects (font (size 1.27 1.27)) hide)
+    )
+    (property "Field4" "IC-08138" (id 4) (at 156.21 104.14 0)
+      (effects (font (size 1.524 1.524)))
+    )
+    (pin "1")
+    (pin "2")
+    (pin "3")
+    (pin "4")
+    (pin "5")
+    (pin "6")
+    (pin "7")
+    (pin "8")
+  )
   (symbol (lib_id "dk_Embedded-Microcontrollers:ATMEGA328P-AU") (at 224.79 64.77 0) (unit 1)
     (in_bom yes) (on_board yes) (fields_autoplaced)
-    (property "Reference" "U?" (id 0) (at 233.68 62.23 0)
+    (property "Reference" "U4" (id 0) (at 233.68 62.23 0)
       (effects (font (size 1.524 1.524)) (justify left))
     )
@@
       (reference "U1") (unit 1) (value "24LC1025") (footprint "Package_SO:SOIC-8_3.9x4.9mm_P1.27mm")
     )
+    (path "/f4ca7441-e845-4bdb-8091-450cec4667dc"
+      (reference "U2") (unit 1) (value "DS1307Z") (footprint "SO08-TIGHT")
+    )
     (path "/cb9194cf-429f-45ca-b70f-daa72d4c7bd0"
-      (reference "U2") (unit 1) (value "24LC1025") (footprint "Package_SO:SOIC-8_3.9x4.9mm_P1.27mm")
+      (reference "U3") (unit 1) (value "24LC1025") (footprint "Package_SO:SOIC-8_3.9x4.9mm_P1.27mm")
     )
     (path "/ff61794e-4165-4898-a842-2e510f945c6f"
-      (reference "U?") (unit 1) (value "ATMEGA328P-AU") (footprint "digikey-footprints:TQFP-32_7x7mm")
+      (reference "U4") (unit 1) (value "ATMEGA328P-AU") (footprint "digikey-footprints:TQFP-32_7x7mm")
     )
     (path "/b0d6e381-d951-43ae-a927-e8561c207b82"

Commit message: added title
Parts:
- U1: footprint (none) -> Package_SO:SOIC-8_3.9x4.9mm_P1.27mm
- Y1: footprint (none) -> Crystal:Crystal_SMD_5032-2Pin_5.0x3.2mm_HandSoldering
Other:
- note added: "MCU Datalogger"
Changed lines of the file:
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@@
     (comment 1 "©2022 by P. CARDON")
+  )
+  (text "MCU Datalogger" (at 22.86 17.78 0)
+    (effects (font (size 1.27 1.27)) (justify left bottom))
   )
   (symbol (lib_id "Device:R") (at 144.78 77.47 0) (unit 1)
@@
     (property "Reference" "Y1" (id 0) (at 138.43 120.65 0))
     (property "Value" "Crystal" (id 1) (at 138.43 123.19 0))
-    (property "Footprint" "" (id 2) (at 138.43 128.27 0)
+    (property "Footprint" "Crystal:Crystal_SMD_5032-2Pin_5.0x3.2mm_HandSoldering" (id 2) (at 138.43 128.27 0)
       (effects (font (size 1.27 1.27)) hide)
     )
@@
       (effects (font (size 1.27 1.27)) (justify left))
     )
-    (property "Footprint" "" (id 2) (at 127 111.76 0)
-      (effects (font (size 1.27 1.27)) hide)
-    )
+    (property "Footprint" "Package_SO:SOIC-8_3.9x4.9mm_P1.27mm" (id 2) (at 127 111.76 0)
+      (effects (font (size 1.27 1.27)) hide)
+    )

Commit message: work in progress
Other:
- title: MCU datalogger -> ${project_name}
Changed lines of the file:
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@@
   (paper "A4")
   (title_block
-    (title "MCU datalogger")
+    (title "${project_name}")
     (date "2022-05-10")
     (rev "${design_version}")

Commit message: Work in progress
Parts:
- removed J1, J3: Conn_01x04_Male, symbol Connector:Conn_01x04_Male
- removed J2: Conn_01x09_Male, symbol Connector:Conn_01x09_Male
- removed J4: Conn_02x03_Odd_Even, symbol Connector_Generic:Conn_02x03_Odd_Even
Other:
- added sheet Connectors (connectors.kicad_sch)
Changed lines of the file:
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@@
     (pin "2")
-  )
-  (symbol (lib_id "Connector:Conn_01x04_Male") (at 110.49 130.81 0) (unit 1)
-    (in_bom yes) (on_board yes) (fields_autoplaced)
-    (property "Reference" "J3" (id 0) (at 111.125 123.19 0))
-    (property "Value" "Conn_01x04_Male" (id 1) (at 111.125 125.73 0))
-    (property "Footprint" "" (id 2) (at 110.49 130.81 0)
-      (effects (font (size 1.27 1.27)) hide)
-    )
-    (property "Datasheet" "~" (id 3) (at 110.49 130.81 0)
-      (effects (font (size 1.27 1.27)) hide)
-    )
-    (pin "1")
-    (pin "2")
-    (pin "3")
-    (pin "4")
   )
   (symbol (lib_id "Mechanical:MountingHole") (at 22.86 133.35 0) (unit 1)
@@
     (pin "1")
     (pin "2")
-  )
-  (symbol (lib_id "Connector:Conn_01x04_Male") (at 64.77 129.54 0) (unit 1)
-    (in_bom yes) (on_board yes) (fields_autoplaced)
-    (property "Reference" "J1" (id 0) (at 65.405 121.92 0))
-    (property "Value" "Conn_01x04_Male" (id 1) (at 65.405 124.46 0))
-    (property "Footprint" "" (id 2) (at 64.77 129.54 0)
-      (effects (font (size 1.27 1.27)) hide)
-    )
-    (property "Datasheet" "~" (id 3) (at 64.77 129.54 0)
-      (effects (font (size 1.27 1.27)) hide)
-    )
-    (pin "1")
-    (pin "2")
-    (pin "3")
-    (pin "4")
   )
   (symbol (lib_id "Device:C") (at 172.72 55.88 0) (unit 1)
@@
     (pin "2")
   )
-  (symbol (lib_id "Connector:Conn_01x09_Male") (at 88.9 138.43 0) (unit 1)
-    (in_bom yes) (on_board yes) (fields_autoplaced)
-    (property "Reference" "J2" (id 0) (at 89.535 123.19 0))
-    (property "Value" "Conn_01x09_Male" (id 1) (at 89.535 125.73 0))
-    (property "Footprint" "" (id 2) (at 88.9 138.43 0)
-      (effects (font (size 1.27 1.27)) hide)
-    )
-    (property "Datasheet" "~" (id 3) (at 88.9 138.43 0)
-      (effects (font (size 1.27 1.27)) hide)
-    )
-    (pin "1")
-    (pin "2")
-    (pin "3")
-    (pin "4")
-    (pin "5")
-    (pin "6")
-    (pin "7")
-    (pin "8")
-    (pin "9")
-  )
   (symbol (lib_id "Mechanical:MountingHole") (at 22.86 119.38 0) (unit 1)
     (in_bom yes) (on_board yes) (fields_autoplaced)
@@
     (pin "1")
     (pin "2")
-  )
-  (symbol (lib_id "Connector_Generic:Conn_02x03_Odd_Even") (at 133.35 140.97 0) (unit 1)
-    (in_bom yes) (on_board yes) (fields_autoplaced)
-    (property "Reference" "J4" (id 0) (at 134.62 132.08 0))
-    (property "Value" "Conn_02x03_Odd_Even" (id 1) (at 134.62 134.62 0))
-    (property "Footprint" "" (id 2) (at 133.35 140.97 0)
-      (effects (font (size 1.27 1.27)) hide)
-    )
-    (property "Datasheet" "~" (id 3) (at 133.35 140.97 0)
-      (effects (font (size 1.27 1.27)) hide)
-    )
-    (pin "1")
-    (pin "2")
-    (pin "3")
-    (pin "4")
-    (pin "5")
-    (pin "6")
   )
   (symbol (lib_id "Device:R") (at 125.73 77.47 0) (unit 1)
@@
     (pin "9")
   )
+  (sheet (at 148.59 171.45) (size 44.45 19.05) (fields_autoplaced)
+    (stroke (width 0.1524) (type solid) (color 0 0 0 0))
+    (fill (color 0 0 0 0.0000))
+    (property "Sheet name" "Connectors" (id 0) (at 148.59 170.7384 0)
+      (effects (font (size 1.27 1.27)) (justify left bottom))
+    )
+    (property "Sheet file" "connectors.kicad_sch" (id 1) (at 148.59 191.0846 0)
+      (effects (font (size 1.27 1.27)) (justify left top))
+    )
+  )
   (sheet_instances
     (path "/" (page "1"))
+    (path "/e171044f-e7d9-47c8-bfac-ea2172ff1f1e" (page "2"))
   )
   (symbol_instances
@@
       (reference "H4") (unit 1) (value "MountingHole") (footprint "")
     )
-    (path "/558d971e-6557-469f-b0ac-2f5f35988e69"
-      (reference "J1") (unit 1) (value "Conn_01x04_Male") (footprint "")
-    )
-    (path "/6cf0b6c9-69cc-4f4b-bdf2-0a012a4f8ec4"
-      (reference "J2") (unit 1) (value "Conn_01x09_Male") (footprint "")
-    )
-    (path "/0c98fa63-4074-4fe2-be93-51eed462d8f7"
-      (reference "J3") (unit 1) (value "Conn_01x04_Male") (footprint "")
-    )
-    (path "/8104d3a9-6cef-467e-99bc-93aa6cf52cb9"
-      (reference "J4") (unit 1) (value "Conn_02x03_Odd_Even") (footprint "")
+    (path "/e171044f-e7d9-47c8-bfac-ea2172ff1f1e/4f1d2a0f-5d3b-4d6a-a2e9-82abd97bddec"
+      (reference "J?") (unit 1) (value "Conn_02x03_Odd_Even") (footprint "")
+    )
+    (path "/e171044f-e7d9-47c8-bfac-ea2172ff1f1e/52b79cd3-0a42-481e-be44-f226ce9de904"
+      (reference "J?") (unit 1) (value "Conn_01x04_Male") (footprint "")
+    )
+    (path "/e171044f-e7d9-47c8-bfac-ea2172ff1f1e/a13d05d7-23de-439d-8aa3-91948a427a90"
+      (reference "J?") (unit 1) (value "Conn_01x04_Male") (footprint "")
+    )
+    (path "/e171044f-e7d9-47c8-bfac-ea2172ff1f1e/d8bcd547-7cd9-464e-a61a-b9901fb48df8"
+      (reference "J?") (unit 1) (value "Conn_01x09_Male") (footprint "")
     )
     (path "/c63b5fc8-661c-44e7-ac4b-00c9fb9e97ae"

Commit message: Work in progress
Other:
- moved on the sheet: BT1, C1, C2, C3, C4, C5, D1, D2, H1, H2, H3, H4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

Commit message: Work in progress
Connections:
- net VCC: now reaches R2.1
- net VCC: now also C1.1, R1.1, U2.8 (VCC)
- net at R2.2: now also U2.7 (SQW)
- net at Y1.1: now also U2.2 (X2)
- net at Y1.2: now also U2.1 (X1)
- net at R1.2: now also U2.3 (VBATT)
- net GND: now reaches C1.2
- net GND: now also U2.4 (GND)
- net SDA: now reaches U2.5 (SDA)
- net SCK: now reaches U2.6 (SCL)
Other:
- note added: "Clock"
- moved on the sheet: BT1, C1, C2, C3, C5, D2, R1, R2, R6, R7, U2, Y1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
