File: My MCU datalogger.kicad_sch (KiCad schematic)
At the start: 25 parts, among them U1 24LC1025, U2 DS1307Z, U3 24LC1025, U4 ATMEGA328P-AU, Y1 Crystal, Y2 Crystal

Commit message: Work in progress
Connections:
- net GND: now also U1.4 (GND), U1.7 (WP), U3.2 (A1), U3.4 (GND), U3.7 (WP)
- net SCK: now also R3.2, U1.6 (SCL), U3.6 (SCL)
- net SDA: now also R4.2, U1.5 (SDA), U3.5 (SDA)
- net VCC: now also R3.1, R4.1, U1.1 (A0), U1.2 (A1), U1.3 (A2), U1.8 (VCC), U3.1 (A0), U3.3 (A2), U3.8 (VCC)
Other:
- note added: "EEPROM"
- note added: "MCU"
- moved on the sheet: R3, R4, U1, U3

Commit message: Finalized schematics
Parts:
- Y2: value Crystal -> 16 MHz
Connections:
- net GND: now also BT1.2 (-), C2.1, C3.1, C4.1, C5.2, R5.1, R7.2, U4.21 (GND), U4.5 (GND)
- net SCK: now also U4.28 (PC5)
- net SDA: now also U4.27 (PC4)
- net VCC: now also R6.1
- net at R7.1: now also D2.1 (K)
- net at C4.2: now also U4.20 (AREF)
- net at C5.1: now also BT1.1 (+), D2.2 (A), U4.18 (AVCC), U4.4 (VCC)
- net at Y2.1: now also C3.2, U4.8 (PB7)
- net at Y2.2: now also C2.2, U4.7 (PB6)
- net RESET: now reaches R6.2
- net RESET: now also U4.29 (PC6)
- net at R5.2: now also D1.1 (K)
- net at D1.2 (A): now also U4.17 (PB5)
- net D3: now reaches U4.1 (PD3)
- net D6: now reaches U4.10 (PD6)
- net D7: now reaches U4.11 (PD7)
- net DB: now reaches U4.12 (PB0)
- net MOSI: now reaches U4.15 (PB3)
- net MISO: now reaches U4.16 (PB4)
- net D4: now reaches U4.2 (PD4)
- net RX: now reaches U4.30 (PD0)
- net TX: now reaches U4.31 (PD1)
- net D2: now reaches U4.32 (PD2)
- net D5: now reaches U4.9 (PD5)
- no-connect marks 0 -> 9
Other:
- sheet Connectors ports: added D2, D3, D4, D5, D6, D7, GND, MISO, MOSI, RESET, RX, SCK, SDA, TX, Vcc; removed none
- moved on the sheet: BT1, C1, C2, C3, C4, C5, D1, D2, R1, R2, R3, R4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

Commit message: Added missing footprints
Parts:
- BT1: footprint (none) -> Connector_PinHeader_2.54mm:PinHeader_1x02_P2.54mm_Vertical
- C1, C2, C3, C4, C5: footprint (none) -> Capacitor_SMD:C_0805_2012Metric
- D1, D2: footprint (none) -> LED_SMD:LED_0805_2012Metric
- H1, H2, H3, H4: footprint (none) -> MountingHole:MountingHole_2.1mm
- R1, R2, R3, R4, R5, R6, R7: footprint (none) -> Resistor_SMD:R_0805_2012Metric
- U2: footprint SO08-TIGHT -> Silicon-Standard:SO08-TIGHT
- Y2: footprint (none) -> Crystal:Crystal_SMD_5032-2Pin_5.0x3.2mm_HandSoldering

Commit message: Fixed ERC errors in schematic
Parts:
- Y1: value Crystal -> 32.768 KHz
Connections:
- net GND: now also U4.3 (GND)
- net VCC: no longer C1.1, R1.1, R2.1, R3.1, R4.1, U1.1 (A0), U1.2 (A1), U1.3 (A2), U1.8 (VCC), U2.8 (VCC), U3.1 (A0), U3.3 (A2), U3.8 (VCC)
- net Vcc: now also BT1.1 (+), C1.1, C5.1, D2.2 (A), R1.1, R2.1, R3.1, R4.1, U1.1 (A0), U1.2 (A1), U1.3 (A2), U1.8 (VCC), U2.8 (VCC), U3.1 (A0), U3.3 (A2), U3.8 (VCC), U4.18 (AVCC), U4.4 (VCC)
Other:
- sheet Connectors ports: added D8; removed none
Changed lines of the file:
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@@
   (no_connect (at 194.31 106.68))
   (no_connect (at 194.31 86.36))
+  (wire (pts (xy 109.22 166.37) (xy 110.49 166.37))
+    (stroke (width 0) (type default) (color 0 0 0 0))
+  )
   (wire (pts (xy 189.23 99.06) (xy 194.31 99.06))
     (stroke (width 0) (type default) (color 0 0 0 0))
@@
     (stroke (width 0) (type default) (color 0 0 0 0))
   )
+  (wire (pts (xy 132.08 168.91) (xy 133.35 168.91))
+    (stroke (width 0) (type default) (color 0 0 0 0))
+  )
   (wire (pts (xy 132.08 63.5) (xy 132.08 78.74))
     (stroke (width 0) (type default) (color 0 0 0 0))
   )
+  (wire (pts (xy 109.22 172.72) (xy 110.49 172.72))
+    (stroke (width 0) (type default) (color 0 0 0 0))
+  )
   (wire (pts (xy 237.49 36.83) (xy 237.49 38.1))
     (stroke (width 0) (type default) (color 0 0 0 0))
@@
     (stroke (width 0) (type default) (color 0 0 0 0))
   )
+  (wire (pts (xy 109.22 175.26) (xy 110.49 175.26))
+    (stroke (width 0) (type default) (color 0 0 0 0))
+  )
   (wire (pts (xy 36.83 111.76) (xy 36.83 116.84))
+    (stroke (width 0) (type default) (color 0 0 0 0))
+  )
+  (wire (pts (xy 132.08 161.29) (xy 133.35 161.29))
     (stroke (width 0) (type default) (color 0 0 0 0))
   )
@@
     (stroke (width 0) (type default) (color 0 0 0 0))
   )
+  (wire (pts (xy 207.01 119.38) (xy 209.55 119.38))
+    (stroke (width 0) (type default) (color 0 0 0 0))
+  )
   (wire (pts (xy 76.2 45.72) (xy 76.2 36.83))
     (stroke (width 0) (type default) (color 0 0 0 0))
@@
     (stroke (width 0) (type default) (color 0 0 0 0))
   )
+  (wire (pts (xy 132.08 171.45) (xy 133.35 171.45))
+    (stroke (width 0) (type default) (color 0 0 0 0))
+  )
   (wire (pts (xy 144.78 48.26) (xy 132.08 48.26))
     (stroke (width 0) (type default) (color 0 0 0 0))
@@
     (stroke (width 0) (type default) (color 0 0 0 0))
   )
+  (wire (pts (xy 109.22 162.56) (xy 110.49 162.56))
+    (stroke (width 0) (type default) (color 0 0 0 0))
+  )
   (wire (pts (xy 189.23 73.66) (xy 194.31 73.66))
     (stroke (width 0) (type default) (color 0 0 0 0))
@@
     (stroke (width 0) (type default) (color 0 0 0 0))
   )
+  (wire (pts (xy 132.08 163.83) (xy 133.35 163.83))
+    (stroke (width 0) (type default) (color 0 0 0 0))
+  )
   (wire (pts (xy 209.55 119.38) (xy 212.09 119.38))
     (stroke (width 0) (type default) (color 0 0 0 0))
   )
+  (wire (pts (xy 109.22 168.91) (xy 110.49 168.91))
+    (stroke (width 0) (type default) (color 0 0 0 0))
+  )
   (wire (pts (xy 46.99 106.68) (xy 49.53 106.68))
     (stroke (width 0) (type default) (color 0 0 0 0))
@@
     (stroke (width 0) (type default) (color 0 0 0 0))
   )
+  (wire (pts (xy 132.08 158.75) (xy 133.35 158.75))
+    (stroke (width 0) (type default) (color 0 0 0 0))
+  )
   (wire (pts (xy 71.12 48.26) (xy 90.17 48.26))
     (stroke (width 0) (type default) (color 0 0 0 0))
@@
   )
   (wire (pts (xy 189.23 60.96) (xy 194.31 60.96))
+    (stroke (width 0) (type default) (color 0 0 0 0))
+  )
+  (wire (pts (xy 109.22 160.02) (xy 110.49 160.02))
     (stroke (width 0) (type default) (color 0 0 0 0))
   )
@@
     (stroke (width 0) (type default) (color 0 0 0 0))
   )
+  (wire (pts (xy 132.08 166.37) (xy 133.35 166.37))
+    (stroke (width 0) (type default) (color 0 0 0 0))
+  )
   (polyline (pts (xy 21.59 88.9) (xy 21.59 129.54))
     (stroke (width 0) (type solid) (color 0 0 0 0))
@@
     (stroke (width 0) (type default) (color 0 0 0 0))
   )
+  (wire (pts (xy 132.08 156.21) (xy 133.35 156.21))
+    (stroke (width 0) (type default) (color 0 0 0 0))
+  )
   (wire (pts (xy 189.23 93.98) (xy 194.31 93.98))
     (stroke (width 0) (type default) (color 0 0 0 0))
   )
   (wire (pts (xy 132.08 63.5) (xy 144.78 63.5))
+    (stroke (width 0) (type default) (color 0 0 0 0))
+  )
+  (wire (pts (xy 109.22 177.8) (xy 110.49 177.8))
     (stroke (width 0) (type default) (color 0 0 0 0))
   )
@@
     (effects (font (size 2 2)) (justify left bottom))
   )
+  (label "MOSI" (at 109.22 177.8 180)
+    (effects (font (size 1.27 1.27)) (justify right bottom))
+  )
   (label "Vcc" (at 102.87 153.67 0)
     (effects (font (size 1.27 1.27)) (justify left bottom))
   )
-  (label "VCC" (at 101.6 92.71 0)
+  (label "Vcc" (at 101.6 92.71 0)
     (effects (font (size 1.27 1.27)) (justify left bottom))
   )
@@
     (effects (font (size 1.27 1.27)) (justify left bottom))
   )
+  (label "RX" (at 109.22 166.37 180)
+    (effects (font (size 1.27 1.27)) (justify right bottom))
+  )
+  (label "SDA" (at 109.22 160.02 180)
+    (effects (font (size 1.27 1.27)) (justify right bottom))
+  )
   (label "SDA" (at 71.12 53.34 0)
     (effects (font (size 1.27 1.27)) (justify left bottom))
@@
     (effects (font (size 1.27 1.27)) (justify left bottom))
   )
-  (label "VCC" (at 55.88 101.6 0)
+  (label "Vcc" (at 55.88 101.6 0)
+    (effects (font (size 1.27 1.27)) (justify left bottom))
+  )
+  (label "D3" (at 133.35 158.75 0)
+    (effects (font (size 1.27 1.27)) (justify left bottom))
+  )
+  (label "D8" (at 133.35 171.45 0)
     (effects (font (size 1.27 1.27)) (justify left bottom))
   )
@@
     (effects (font (size 1.27 1.27)) (justify left bottom))
   )
-  (label "VCC" (at 69.85 92.71 0)
+  (label "Vcc" (at 69.85 92.71 0)
     (effects (font (size 1.27 1.27)) (justify left bottom))
   )
@@
     (effects (font (size 1.27 1.27)) (justify left bottom))
   )
+  (label "D5" (at 133.35 163.83 0)
+    (effects (font (size 1.27 1.27)) (justify left bottom))
+  )
+  (label "SCK" (at 109.22 162.56 180)
+    (effects (font (size 1.27 1.27)) (justify right bottom))
+  )
   (label "D3" (at 189.23 48.26 0)
     (effects (font (size 1.27 1.27)) (justify left bottom))
   )
-  (label "VCC" (at 55.88 106.68 0)
-    (effects (font (size 1.27 1.27)) (justify left bottom))
-  )
-  (label "VCC" (at 36.83 92.71 0)
-    (effects (font (size 1.27 1.27)) (justify left bottom))
-  )
-  (label "VCC" (at 22.86 106.68 0)
+  (label "Vcc" (at 55.88 106.68 0)
+    (effects (font (size 1.27 1.27)) (justify left bottom))
+  )
+  (label "Vcc" (at 36.83 92.71 0)
+    (effects (font (size 1.27 1.27)) (justify left bottom))
+  )
+  (label "D7" (at 133.35 168.91 0)
+    (effects (font (size 1.27 1.27)) (justify left bottom))
+  )
+  (label "Vcc" (at 22.86 106.68 0)
     (effects (font (size 1.27 1.27)) (justify left bottom))
   )
@@
     (effects (font (size 1.27 1.27)) (justify left bottom))
   )
-  (label "VCC" (at 81.28 33.02 0)
+  (label "D2" (at 133.35 156.21 0)
+    (effects (font (size 1.27 1.27)) (justify left bottom))
+  )
+  (label "Vcc" (at 81.28 33.02 0)
     (effects (font (size 1.27 1.27)) (justify left bottom))
   )
@@
     (effects (font (size 1.27 1.27)) (justify left bottom))
   )
-  (label "VCC" (at 22.86 101.6 0)
+  (label "D6" (at 133.35 166.37 0)
+    (effects (font (size 1.27 1.27)) (justify left bottom))
+  )
+  (label "Vcc" (at 22.86 101.6 0)
+    (effects (font (size 1.27 1.27)) (justify left bottom))
+  )
+  (label "MISO" (at 109.22 172.72 180)
+    (effects (font (size 1.27 1.27)) (justify right bottom))
+  )
+  (label "RESET" (at 109.22 175.26 180)
+    (effects (font (size 1.27 1.27)) (justify right bottom))
+  )
+  (label "Vcc" (at 224.79 38.1 0)
     (effects (font (size 1.27 1.27)) (justify left bottom))
   )
@@
     (effects (font (size 1.27 1.27)) (justify left bottom))
   )
+  (label "D4" (at 133.35 161.29 0)
+    (effects (font (size 1.27 1.27)) (justify left bottom))
+  )
   (label "SDA" (at 48.26 101.6 0)
     (effects (font (size 1.27 1.27)) (justify left bottom))
   )
+  (label "TX" (at 109.22 168.91 180)
+    (effects (font (size 1.27 1.27)) (justify right bottom))
+  )
   (label "TX" (at 189.23 101.6 0)
     (effects (font (size 1.27 1.27)) (justify left bottom))
@@
     (effects (font (size 1.27 1.27)) (justify left bottom))
   )
-  (label "VCC" (at 22.86 104.14 0)
+  (label "Vcc" (at 22.86 104.14 0)
     (effects (font (size 1.27 1.27)) (justify left bottom))
   )
@@
   )
   (symbol (lib_id "Device:Crystal") (at 27.94 49.53 90) (unit 1)
-    (in_bom yes) (on_board yes) (fields_autoplaced)
-    (property "Reference" "Y1" (id 0) (at 31.75 48.2599 90)
+    (in_bom yes) (on_board yes)
+    (property "Reference" "Y1" (id 0) (at 24.13 41.91 90)
       (effects (font (size 1.27 1.27)) (justify right))
     )
-    (property "Value" "Crystal" (id 1) (at 31.75 50.7999 90)
+    (property "Value" "32.768 KHz" (id 1) (at 24.13 44.45 90)
       (effects (font (size 1.27 1.27)) (justify right))
     )
@@
       (effects (font (size 1.27 1.27)) (justify right))
     )
+    (pin "D8" bidirectional (at 132.08 171.45 0)
+      (effects (font (size 1.27 1.27)) (justify right))
+    )
   )
   (sheet_instances
@@
     )
     (path "/b0d6e381-d951-43ae-a927-e8561c207b82"
-      (reference "Y1") (unit 1) (value "Crystal") (footprint "Crystal:Crystal_SMD_5032-2Pin_5.0x3.2mm_HandSoldering")
+      (reference "Y1") (unit 1) (value "32.768 KHz") (footprint "Crystal:Crystal_SMD_5032-2Pin_5.0x3.2mm_HandSoldering")
     )
     (path "/6256d3e5-5699-458b-966c-c925c4481fa4"

Commit message: Various fixes
Other:
- note added: "Mounting holes"
- moved on the sheet: H1, H2, H3, H4
Changed lines of the file:
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@@
     (stroke (width 0) (type default) (color 0 0 0 0))
+  )
+  (polyline (pts (xy 163.83 151.13) (xy 190.5 151.13))
+    (stroke (width 0) (type solid) (color 0 0 0 0))
   )
   (wire (pts (xy 166.37 48.26) (xy 166.37 52.07))
@@
     (stroke (width 0) (type default) (color 0 0 0 0))
   )
+  (polyline (pts (xy 190.5 180.34) (xy 163.83 180.34))
+    (stroke (width 0) (type solid) (color 0 0 0 0))
+  )
   (wire (pts (xy 45.72 58.42) (xy 45.72 50.8))
     (stroke (width 0) (type default) (color 0 0 0 0))
@@
     (stroke (width 0) (type default) (color 0 0 0 0))
   )
+  (polyline (pts (xy 190.5 151.13) (xy 190.5 180.34))
+    (stroke (width 0) (type solid) (color 0 0 0 0))
+  )
   (wire (pts (xy 269.24 81.28) (xy 269.24 120.65))
     (stroke (width 0) (type default) (color 0 0 0 0))
@@
   (wire (pts (xy 71.12 48.26) (xy 90.17 48.26))
     (stroke (width 0) (type default) (color 0 0 0 0))
+  )
+  (polyline (pts (xy 163.83 151.13) (xy 163.83 180.34))
+    (stroke (width 0) (type solid) (color 0 0 0 0))
   )
   (wire (pts (xy 49.53 106.68) (xy 49.53 116.84))
@@
     (effects (font (size 2 2)) (justify left bottom))
   )
+  (text "Mounting holes\n" (at 163.83 149.86 0)
+    (effects (font (size 2 2)) (justify left bottom))
+  )
   (label "MOSI" (at 109.22 177.8 180)
     (effects (font (size 1.27 1.27)) (justify right bottom))
@@
     (pin "1")
   )
-  (symbol (lib_id "Mechanical:MountingHole") (at 182.88 193.04 0) (unit 1)
-    (in_bom yes) (on_board yes) (fields_autoplaced)
-    (property "Reference" "H4" (id 0) (at 185.42 191.7699 0)
-      (effects (font (size 1.27 1.27)) (justify left))
-    )
-    (property "Value" "MountingHole" (id 1) (at 185.42 194.3099 0)
-      (effects (font (size 1.27 1.27)) (justify left))
-    )
-    (property "Footprint" "MountingHole:MountingHole_2.1mm" (id 2) (at 182.88 193.04 0)
-      (effects (font (size 1.27 1.27)) hide)
-    )
-    (property "Datasheet" "~" (id 3) (at 182.88 193.04 0)
+  (symbol (lib_id "Mechanical:MountingHole") (at 167.64 173.99 0) (unit 1)
+    (in_bom yes) (on_board yes) (fields_autoplaced)
+    (property "Reference" "H4" (id 0) (at 170.18 172.7199 0)
+      (effects (font (size 1.27 1.27)) (justify left))
+    )
+    (property "Value" "MountingHole" (id 1) (at 170.18 175.2599 0)
+      (effects (font (size 1.27 1.27)) (justify left))
+    )
+    (property "Footprint" "MountingHole:MountingHole_2.1mm" (id 2) (at 167.64 173.99 0)
+      (effects (font (size 1.27 1.27)) hide)
+    )
+    (property "Datasheet" "~" (id 3) (at 167.64 173.99 0)
       (effects (font (size 1.27 1.27)) hide)
     )
@@
     (pin "2")
   )
-  (symbol (lib_id "Mechanical:MountingHole") (at 182.88 179.07 0) (unit 1)
-    (in_bom yes) (on_board yes) (fields_autoplaced)
-    (property "Reference" "H2" (id 0) (at 185.42 177.7999 0)
-      (effects (font (size 1.27 1.27)) (justify left))
-    )
-    (property "Value" "MountingHole" (id 1) (at 185.42 180.3399 0)
-      (effects (font (size 1.27 1.27)) (justify left))
-    )
-    (property "Footprint" "MountingHole:MountingHole_2.1mm" (id 2) (at 182.88 179.07 0)
-      (effects (font (size 1.27 1.27)) hide)
-    )
-    (property "Datasheet" "~" (id 3) (at 182.88 179.07 0)
+  (symbol (lib_id "Mechanical:MountingHole") (at 167.64 160.02 0) (unit 1)
+    (in_bom yes) (on_board yes) (fields_autoplaced)
+    (property "Reference" "H2" (id 0) (at 170.18 158.7499 0)
+      (effects (font (size 1.27 1.27)) (justify left))
+    )
+    (property "Value" "MountingHole" (id 1) (at 170.18 161.2899 0)
+      (effects (font (size 1.27 1.27)) (justify left))
+    )
+    (property "Footprint" "MountingHole:MountingHole_2.1mm" (id 2) (at 167.64 160.02 0)
+      (effects (font (size 1.27 1.27)) hide)
+    )
+    (property "Datasheet" "~" (id 3) (at 167.64 160.02 0)
       (effects (font (size 1.27 1.27)) hide)
     )
@@
     (pin "2")
   )
-  (symbol (lib_id "Mechanical:MountingHole") (at 182.88 172.72 0) (unit 1)
-    (in_bom yes) (on_board yes) (fields_autoplaced)
-    (property "Reference" "H1" (id 0) (at 185.42 171.4499 0)
-      (effects (font (size 1.27 1.27)) (justify left))
-    )
-    (property "Value" "MountingHole" (id 1) (at 185.42 173.9899 0)
-      (effects (font (size 1.27 1.27)) (justify left))
-    )
-    (property "Footprint" "MountingHole:MountingHole_2.1mm" (id 2) (at 182.88 172.72 0)
-      (effects (font (size 1.27 1.27)) hide)
-    )
-    (property "Datasheet" "~" (id 3) (at 182.88 172.72 0)
+  (symbol (lib_id "Mechanical:MountingHole") (at 167.64 153.67 0) (unit 1)
+    (in_bom yes) (on_board yes) (fields_autoplaced)
+    (property "Reference" "H1" (id 0) (at 170.18 152.3999 0)
+      (effects (font (size 1.27 1.27)) (justify left))
+    )
+    (property "Value" "MountingHole" (id 1) (at 170.18 154.9399 0)
+      (effects (font (size 1.27 1.27)) (justify left))
+    )
+    (property "Footprint" "MountingHole:MountingHole_2.1mm" (id 2) (at 167.64 153.67 0)
+      (effects (font (size 1.27 1.27)) hide)
+    )
+    (property "Datasheet" "~" (id 3) (at 167.64 153.67 0)
       (effects (font (size 1.27 1.27)) hide)
     )
@@
     (pin "8")
   )
-  (symbol (lib_id "Mechanical:MountingHole") (at 182.88 185.42 0) (unit 1)
-    (in_bom yes) (on_board yes) (fields_autoplaced)
-    (property "Reference" "H3" (id 0) (at 185.42 184.1499 0)
-      (effects (font (size 1.27 1.27)) (justify left))
-    )
-    (property "Value" "MountingHole" (id 1) (at 185.42 186.6899 0)
-      (effects (font (size 1.27 1.27)) (justify left))
-    )
-    (property "Footprint" "MountingHole:MountingHole_2.1mm" (id 2) (at 182.88 185.42 0)
-      (effects (font (size 1.27 1.27)) hide)
-    )
-    (property "Datasheet" "~" (id 3) (at 182.88 185.42 0)
-      (effects (font (size 1.27 1.27)) hide)
-    )
+  (symbol (lib_id "Mechanical:MountingHole") (at 167.64 166.37 0) (unit 1)
+    (in_bom yes) (on_board yes) (fields_autoplaced)
+    (property "Reference" "H3" (id 0) (at 170.18 165.0999 0)
+      (effects (font (size 1.27 1.27)) (justify left))
+    )
+    (property "Value" "MountingHole" (id 1) (at 170.18 167.6399 0)
+      (effects (font (size 1.27 1.27)) (justify left))
+    )
+    (property "Footprint" "MountingHole:MountingHole_2.1mm" (id 2) (at 167.64 166.37 0)
+      (effects (font (size 1.27 1.27)) hide)
+    )
+    (property "Datasheet" "~" (id 3) (at 167.64 166.37 0)
+      (effects (font (size 1.27 1.27)) hide)
+    )
