File: My MCU datalogger.kicad_sch (KiCad schematic)
At the start: 25 parts, among them U1 24LC1025, U2 DS1307Z, U3 24LC1025, U4 ATMEGA328P-AU, Y1 32.768 KHz, Y2 16 MHz

Commit message: Various refinements
Connections:
- net VCC is gone; now on net Vcc: R6.1
Other:
- moved on the sheet: H1, H2, H3, H4
Changed lines of the file:
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@@
   )
   (text "EEPROM" (at 22.86 87.63 0)
-    (effects (font (size 2 2)) (justify left bottom))
+    (effects (font (size 2 2) (thickness 0.4) bold) (justify left bottom))
   )
   (text "MCU" (at 125.73 27.94 0)
-    (effects (font (size 2 2)) (justify left bottom))
+    (effects (font (size 2 2) (thickness 0.4) bold) (justify left bottom))
   )
   (text "MCU Datalogger" (at 121.92 21.59 0)
@@
   )
   (text "Clock" (at 22.86 27.94 0)
-    (effects (font (size 2 2)) (justify left bottom))
+    (effects (font (size 2 2) (thickness 0.4) bold) (justify left bottom))
   )
   (text "Mounting holes\n" (at 163.83 149.86 0)
-    (effects (font (size 2 2)) (justify left bottom))
+    (effects (font (size 2 2) (thickness 0.4) bold) (justify left bottom))
   )
   (label "MOSI" (at 109.22 177.8 180)
@@
     (effects (font (size 1.27 1.27)) (justify left bottom))
   )
-  (label "VCC" (at 158.75 96.52 0)
+  (label "Vcc" (at 158.75 96.52 0)
     (effects (font (size 1.27 1.27)) (justify left bottom))
   )
@@
     (pin "1")
   )
-  (symbol (lib_id "Mechanical:MountingHole") (at 167.64 173.99 0) (unit 1)
-    (in_bom yes) (on_board yes) (fields_autoplaced)
-    (property "Reference" "H4" (id 0) (at 170.18 172.7199 0)
-      (effects (font (size 1.27 1.27)) (justify left))
-    )
-    (property "Value" "MountingHole" (id 1) (at 170.18 175.2599 0)
-      (effects (font (size 1.27 1.27)) (justify left))
-    )
-    (property "Footprint" "MountingHole:MountingHole_2.1mm" (id 2) (at 167.64 173.99 0)
-      (effects (font (size 1.27 1.27)) hide)
-    )
-    (property "Datasheet" "~" (id 3) (at 167.64 173.99 0)
+  (symbol (lib_id "Mechanical:MountingHole") (at 170.18 175.26 0) (unit 1)
+    (in_bom yes) (on_board yes) (fields_autoplaced)
+    (property "Reference" "H4" (id 0) (at 172.72 173.9899 0)
+      (effects (font (size 1.27 1.27)) (justify left))
+    )
+    (property "Value" "MountingHole" (id 1) (at 172.72 176.5299 0)
+      (effects (font (size 1.27 1.27)) (justify left))
+    )
+    (property "Footprint" "MountingHole:MountingHole_2.1mm" (id 2) (at 170.18 175.26 0)
+      (effects (font (size 1.27 1.27)) hide)
+    )
+    (property "Datasheet" "~" (id 3) (at 170.18 175.26 0)
       (effects (font (size 1.27 1.27)) hide)
     )
@@
     (pin "2")
   )
-  (symbol (lib_id "Mechanical:MountingHole") (at 167.64 160.02 0) (unit 1)
-    (in_bom yes) (on_board yes) (fields_autoplaced)
-    (property "Reference" "H2" (id 0) (at 170.18 158.7499 0)
-      (effects (font (size 1.27 1.27)) (justify left))
-    )
-    (property "Value" "MountingHole" (id 1) (at 170.18 161.2899 0)
-      (effects (font (size 1.27 1.27)) (justify left))
-    )
-    (property "Footprint" "MountingHole:MountingHole_2.1mm" (id 2) (at 167.64 160.02 0)
-      (effects (font (size 1.27 1.27)) hide)
-    )
-    (property "Datasheet" "~" (id 3) (at 167.64 160.02 0)
+  (symbol (lib_id "Mechanical:MountingHole") (at 170.18 162.56 0) (unit 1)
+    (in_bom yes) (on_board yes) (fields_autoplaced)
+    (property "Reference" "H2" (id 0) (at 172.72 161.2899 0)
+      (effects (font (size 1.27 1.27)) (justify left))
+    )
+    (property "Value" "MountingHole" (id 1) (at 172.72 163.8299 0)
+      (effects (font (size 1.27 1.27)) (justify left))
+    )
+    (property "Footprint" "MountingHole:MountingHole_2.1mm" (id 2) (at 170.18 162.56 0)
+      (effects (font (size 1.27 1.27)) hide)
+    )
+    (property "Datasheet" "~" (id 3) (at 170.18 162.56 0)
       (effects (font (size 1.27 1.27)) hide)
     )
@@
     (pin "2")
   )
-  (symbol (lib_id "Mechanical:MountingHole") (at 167.64 153.67 0) (unit 1)
-    (in_bom yes) (on_board yes) (fields_autoplaced)
-    (property "Reference" "H1" (id 0) (at 170.18 152.3999 0)
-      (effects (font (size 1.27 1.27)) (justify left))
-    )
-    (property "Value" "MountingHole" (id 1) (at 170.18 154.9399 0)
-      (effects (font (size 1.27 1.27)) (justify left))
-    )
-    (property "Footprint" "MountingHole:MountingHole_2.1mm" (id 2) (at 167.64 153.67 0)
-      (effects (font (size 1.27 1.27)) hide)
-    )
-    (property "Datasheet" "~" (id 3) (at 167.64 153.67 0)
+  (symbol (lib_id "Mechanical:MountingHole") (at 170.18 156.21 0) (unit 1)
+    (in_bom yes) (on_board yes) (fields_autoplaced)
+    (property "Reference" "H1" (id 0) (at 172.72 154.9399 0)
+      (effects (font (size 1.27 1.27)) (justify left))
+    )
+    (property "Value" "MountingHole" (id 1) (at 172.72 157.4799 0)
+      (effects (font (size 1.27 1.27)) (justify left))
+    )
+    (property "Footprint" "MountingHole:MountingHole_2.1mm" (id 2) (at 170.18 156.21 0)
+      (effects (font (size 1.27 1.27)) hide)
+    )
+    (property "Datasheet" "~" (id 3) (at 170.18 156.21 0)
       (effects (font (size 1.27 1.27)) hide)
     )
@@
   )
   (symbol (lib_id "Memory_EEPROM:24LC1025") (at 36.83 104.14 0) (unit 1)
-    (in_bom yes) (on_board yes) (fields_autoplaced)
-    (property "Reference" "U1" (id 0) (at 38.8494 93.98 0)
-      (effects (font (size 1.27 1.27)) (justify left))
-    )
-    (property "Value" "24LC1025" (id 1) (at 38.8494 96.52 0)
+    (in_bom yes) (on_board yes)
+    (property "Reference" "U1" (id 0) (at 25.4 91.44 0)
+      (effects (font (size 1.27 1.27)) (justify left))
+    )
+    (property "Value" "24LC1025" (id 1) (at 25.4 93.98 0)
       (effects (font (size 1.27 1.27)) (justify left))
     )
@@
     (pin "8")
   )
-  (symbol (lib_id "Mechanical:MountingHole") (at 167.64 166.37 0) (unit 1)
-    (in_bom yes) (on_board yes) (fields_autoplaced)
-    (property "Reference" "H3" (id 0) (at 170.18 165.0999 0)
-      (effects (font (size 1.27 1.27)) (justify left))
-    )
-    (property "Value" "MountingHole" (id 1) (at 170.18 167.6399 0)
-      (effects (font (size 1.27 1.27)) (justify left))
-    )
-    (property "Footprint" "MountingHole:MountingHole_2.1mm" (id 2) (at 167.64 166.37 0)
-      (effects (font (size 1.27 1.27)) hide)
-    )
-    (property "Datasheet" "~" (id 3) (at 167.64 166.37 0)
+  (symbol (lib_id "Mechanical:MountingHole") (at 170.18 168.91 0) (unit 1)
+    (in_bom yes) (on_board yes) (fields_autoplaced)
+    (property "Reference" "H3" (id 0) (at 172.72 167.6399 0)
+      (effects (font (size 1.27 1.27)) (justify left))
+    )
+    (property "Value" "MountingHole" (id 1) (at 172.72 170.1799 0)
+      (effects (font (size 1.27 1.27)) (justify left))
+    )
+    (property "Footprint" "MountingHole:MountingHole_2.1mm" (id 2) (at 170.18 168.91 0)
+      (effects (font (size 1.27 1.27)) hide)
+    )
+    (property "Datasheet" "~" (id 3) (at 170.18 168.91 0)
       (effects (font (size 1.27 1.27)) hide)
     )
@@
   )
   (symbol (lib_id "Memory_EEPROM:24LC1025") (at 69.85 104.14 0) (unit 1)
-    (in_bom yes) (on_board yes) (fields_autoplaced)
-    (property "Reference" "U3" (id 0) (at 71.8694 93.98 0)
-      (effects (font (size 1.27 1.27)) (justify left))
-    )
-    (property "Value" "24LC1025" (id 1) (at 71.8694 96.52 0)
+    (in_bom yes) (on_board yes)
+    (property "Reference" "U3" (id 0) (at 58.42 91.44 0)
+      (effects (font (size 1.27 1.27)) (justify left))
+    )
+    (property "Value" "24LC1025" (id 1) (at 58.42 93.98 0)
       (effects (font (size 1.27 1.27)) (justify left))
     )
@@
     (fill (color 0 0 0 0.0000))
     (property "Sheet name" "Connectors" (id 0) (at 110.49 150.4184 0)
-      (effects (font (size 2 2)) (justify left bottom))
+      (effects (font (size 2 2) bold) (justify left bottom))
     )
     (property "Sheet file" "connectors.kicad_sch" (id 1) (at 107.95 181.61 0)

Commit message: Final outline
Connections:
- net DB is gone; now on net D8: U4.12 (PB0)
Changed lines of the file:
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@@
     (effects (font (size 1.27 1.27)) (justify left bottom))
   )
-  (label "DB" (at 189.23 66.04 0)
+  (label "D8" (at 189.23 66.04 0)
     (effects (font (size 1.27 1.27)) (justify left bottom))
   )
