File: connectors.kicad_sch (KiCad schematic)
At the start: 4 parts

Commit message: Work in progress
Parts:
- gave numbers to parts that had none: 4
Changed lines of the file:
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@@
   (symbol (lib_id "Connector_Generic:Conn_02x03_Odd_Even") (at 167.64 86.36 0) (unit 1)
     (in_bom yes) (on_board yes)
-    (property "Reference" "J?" (id 0) (at 168.91 77.47 0))
+    (property "Reference" "J4" (id 0) (at 168.91 77.47 0))
     (property "Value" "Conn_02x03_Odd_Even" (id 1) (at 168.91 80.01 0))
     (property "Footprint" "" (id 2) (at 167.64 86.36 0)
@@
   (symbol (lib_id "Connector:Conn_01x04_Male") (at 95.25 83.82 0) (unit 1)
     (in_bom yes) (on_board yes) (fields_autoplaced)
-    (property "Reference" "J?" (id 0) (at 95.885 76.2 0))
+    (property "Reference" "J1" (id 0) (at 95.885 76.2 0))
     (property "Value" "Conn_01x04_Male" (id 1) (at 95.885 78.74 0))
     (property "Footprint" "" (id 2) (at 95.25 83.82 0)
@@
   (symbol (lib_id "Connector:Conn_01x04_Male") (at 140.97 85.09 0) (unit 1)
     (in_bom yes) (on_board yes) (fields_autoplaced)
-    (property "Reference" "J?" (id 0) (at 141.605 77.47 0))
+    (property "Reference" "J3" (id 0) (at 141.605 77.47 0))
     (property "Value" "Conn_01x04_Male" (id 1) (at 141.605 80.01 0))
     (property "Footprint" "" (id 2) (at 140.97 85.09 0)
@@
   (symbol (lib_id "Connector:Conn_01x09_Male") (at 119.38 92.71 0) (unit 1)
     (in_bom yes) (on_board yes) (fields_autoplaced)
-    (property "Reference" "J?" (id 0) (at 120.015 77.47 0))
+    (property "Reference" "J2" (id 0) (at 120.015 77.47 0))
     (property "Value" "Conn_01x09_Male" (id 1) (at 120.015 80.01 0))
     (property "Footprint" "" (id 2) (at 119.38 92.71 0)

Commit message: Finalized schematics
Connections:
- net MISO: now reaches J4.1 (Pin_1)
- net Vcc: now reaches J4.2 (Pin_2)
- net Vcc: now also J1.2 (Pin_2), J2.9 (Pin_9), J3.2 (Pin_2)
- net SCK: now reaches J4.3 (Pin_3)
- net SCK: now also J1.4 (Pin_4)
- net MOSI: now reaches J4.4 (Pin_4)
- net RESET: now reaches J4.5 (Pin_5)
- net GND: now reaches J4.6 (Pin_6)
- net GND: now also J1.1 (Pin_1), J2.8 (Pin_8), J3.1 (Pin_1)
- net SDA: now reaches J1.3 (Pin_3)
- net RX: now reaches J3.3 (Pin_3)
- net TX: now reaches J3.4 (Pin_4)
- net D2: now reaches J2.1 (Pin_1)
- net D3: now reaches J2.2 (Pin_2)
- net D4: now reaches J2.3 (Pin_3)
- net D5: now reaches J2.4 (Pin_4)
- net D6: now reaches J2.5 (Pin_5)
- net D7: now reaches J2.6 (Pin_6)
- net D8: now reaches J2.7 (Pin_7)
Other:
- note added: "GPIO"
- note added: "I2C"
- note added: "ICSP"
- note added: "Serial UART"
Changed lines of the file:
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@@
 (kicad_sch (version 20211123) (generator eeschema)
   (paper "A4")
+  (text "I2C" (at 97.79 95.25 0)
+    (effects (font (size 2 2)) (justify left bottom))
+  )
+  (text "Serial UART" (at 134.62 95.25 0)
+    (effects (font (size 2 2)) (justify left bottom))
+  )
+  (text "GPIO" (at 120.65 107.95 0)
+    (effects (font (size 2 2)) (justify left bottom))
+  )
+  (text "ICSP" (at 166.37 95.25 0)
+    (effects (font (size 2 2)) (justify left bottom))
+  )
+  (hierarchical_label "GND" (shape passive) (at 124.46 100.33 0)
+    (effects (font (size 1.27 1.27)) (justify left))
+  )
+  (hierarchical_label "RX" (shape input) (at 146.05 87.63 0)
+    (effects (font (size 1.27 1.27)) (justify left))
+  )
+  (hierarchical_label "Vcc" (shape passive) (at 146.05 85.09 0)
+    (effects (font (size 1.27 1.27)) (justify left))
+  )
+  (hierarchical_label "SCK" (shape passive) (at 100.33 88.9 0)
+    (effects (font (size 1.27 1.27)) (justify left))
+  )
+  (hierarchical_label "D8" (shape bidirectional) (at 124.46 97.79 0)
+    (effects (font (size 1.27 1.27)) (justify left))
+  )
+  (hierarchical_label "SCK" (shape passive) (at 162.56 86.36 180)
+    (effects (font (size 1.27 1.27)) (justify right))
+  )
+  (hierarchical_label "D7" (shape bidirectional) (at 124.46 95.25 0)
+    (effects (font (size 1.27 1.27)) (justify left))
+  )
+  (hierarchical_label "GND" (shape passive) (at 146.05 82.55 0)
+    (effects (font (size 1.27 1.27)) (justify left))
+  )
+  (hierarchical_label "GND" (shape passive) (at 175.26 88.9 0)
+    (effects (font (size 1.27 1.27)) (justify left))
+  )
+  (hierarchical_label "D4" (shape bidirectional) (at 124.46 87.63 0)
+    (effects (font (size 1.27 1.27)) (justify left))
+  )
+  (hierarchical_label "D6" (shape bidirectional) (at 124.46 92.71 0)
+    (effects (font (size 1.27 1.27)) (justify left))
+  )
+  (hierarchical_label "RESET" (shape passive) (at 162.56 88.9 180)
+    (effects (font (size 1.27 1.27)) (justify right))
+  )
+  (hierarchical_label "D3" (shape bidirectional) (at 124.46 85.09 0)
+    (effects (font (size 1.27 1.27)) (justify left))
+  )
+  (hierarchical_label "MOSI" (shape input) (at 175.26 86.36 0)
+    (effects (font (size 1.27 1.27)) (justify left))
+  )
+  (hierarchical_label "Vcc" (shape passive) (at 124.46 102.87 0)
+    (effects (font (size 1.27 1.27)) (justify left))
+  )
+  (hierarchical_label "D2" (shape bidirectional) (at 124.46 82.55 0)
+    (effects (font (size 1.27 1.27)) (justify left))
+  )
+  (hierarchical_label "Vcc" (shape passive) (at 100.33 83.82 0)
+    (effects (font (size 1.27 1.27)) (justify left))
+  )
+  (hierarchical_label "D5" (shape bidirectional) (at 124.46 90.17 0)
+    (effects (font (size 1.27 1.27)) (justify left))
+  )
+  (hierarchical_label "MISO" (shape output) (at 162.56 83.82 180)
+    (effects (font (size 1.27 1.27)) (justify right))
+  )
+  (hierarchical_label "GND" (shape passive) (at 100.33 81.28 0)
+    (effects (font (size 1.27 1.27)) (justify left))
+  )
+  (hierarchical_label "SDA" (shape bidirectional) (at 100.33 86.36 0)
+    (effects (font (size 1.27 1.27)) (justify left))
+  )
+  (hierarchical_label "TX" (shape output) (at 146.05 90.17 0)
+    (effects (font (size 1.27 1.27)) (justify left))
+  )
+  (hierarchical_label "Vcc" (shape passive) (at 175.26 83.82 0)
+    (effects (font (size 1.27 1.27)) (justify left))
+  )
   (symbol (lib_id "Connector_Generic:Conn_02x03_Odd_Even") (at 167.64 86.36 0) (unit 1)
     (in_bom yes) (on_board yes)

Commit message: Added missing footprints
Parts:
- J1, J3: footprint (none) -> Connector_PinHeader_2.54mm:PinHeader_1x04_P2.54mm_Vertical
- J2, J4: footprint (none) -> Connector_PinHeader_2.54mm:PinHeader_1x09_P2.54mm_Vertical
Changed lines of the file:
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@@
     (property "Reference" "J4" (id 0) (at 168.91 77.47 0))
     (property "Value" "Conn_02x03_Odd_Even" (id 1) (at 168.91 80.01 0))
-    (property "Footprint" "" (id 2) (at 167.64 86.36 0)
+    (property "Footprint" "Connector_PinHeader_2.54mm:PinHeader_1x09_P2.54mm_Vertical" (id 2) (at 167.64 86.36 0)
       (effects (font (size 1.27 1.27)) hide)
     )
@@
     (property "Reference" "J1" (id 0) (at 95.885 76.2 0))
     (property "Value" "Conn_01x04_Male" (id 1) (at 95.885 78.74 0))
-    (property "Footprint" "" (id 2) (at 95.25 83.82 0)
+    (property "Footprint" "Connector_PinHeader_2.54mm:PinHeader_1x04_P2.54mm_Vertical" (id 2) (at 95.25 83.82 0)
       (effects (font (size 1.27 1.27)) hide)
     )
@@
     (property "Reference" "J3" (id 0) (at 141.605 77.47 0))
     (property "Value" "Conn_01x04_Male" (id 1) (at 141.605 80.01 0))
-    (property "Footprint" "" (id 2) (at 140.97 85.09 0)
+    (property "Footprint" "Connector_PinHeader_2.54mm:PinHeader_1x04_P2.54mm_Vertical" (id 2) (at 140.97 85.09 0)
       (effects (font (size 1.27 1.27)) hide)
     )
@@
     (property "Reference" "J2" (id 0) (at 120.015 77.47 0))
     (property "Value" "Conn_01x09_Male" (id 1) (at 120.015 80.01 0))
-    (property "Footprint" "" (id 2) (at 119.38 92.71 0)
+    (property "Footprint" "Connector_PinHeader_2.54mm:PinHeader_1x09_P2.54mm_Vertical" (id 2) (at 119.38 92.71 0)
       (effects (font (size 1.27 1.27)) hide)
     )

Commit message: Various fixes
Other:
- note added: "Connectors"
- company: (none) -> PC Soft War
- title: (none) -> Connectors
- moved on the sheet: J1, J2, J3, J4
Changed lines of the file:
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@@
 (kicad_sch (version 20211123) (generator eeschema)
-  (paper "A4")
-  (text "I2C" (at 97.79 95.25 0)
+  (paper "A5")
+  (title_block
+    (title "Connectors")
+    (date "2022-05-12")
+    (rev "${design_version}")
+    (company "PC Soft War")
+    (comment 1 "©2022 by P. CARDON")
+  )
+  (polyline (pts (xy 63.5 25.4) (xy 63.5 101.6))
+    (stroke (width 0) (type solid) (color 0 0 0 0))
+  )
+  (polyline (pts (xy 63.5 101.6) (xy 63.5 101.6))
+    (stroke (width 0) (type default) (color 0 0 0 0))
+  )
+  (polyline (pts (xy 139.7 25.4) (xy 139.7 101.6))
+    (stroke (width 0) (type solid) (color 0 0 0 0))
+  )
+  (polyline (pts (xy 63.5 25.4) (xy 139.7 25.4))
+    (stroke (width 0) (type solid) (color 0 0 0 0))
+  )
+  (polyline (pts (xy 63.5 101.6) (xy 139.7 101.6))
+    (stroke (width 0) (type solid) (color 0 0 0 0))
+  )
+  (text "Connectors" (at 63.5 24.13 0)
     (effects (font (size 2 2)) (justify left bottom))
   )
-  (text "Serial UART" (at 134.62 95.25 0)
+  (text "I2C" (at 78.74 52.07 0)
     (effects (font (size 2 2)) (justify left bottom))
   )
-  (text "GPIO" (at 120.65 107.95 0)
+  (text "Serial UART" (at 114.3 50.8 0)
     (effects (font (size 2 2)) (justify left bottom))
   )
-  (text "ICSP" (at 166.37 95.25 0)
+  (text "GPIO" (at 96.52 138.43 0)
     (effects (font (size 2 2)) (justify left bottom))
   )
-  (hierarchical_label "GND" (shape passive) (at 124.46 100.33 0)
+  (text "ICSP" (at 119.38 82.55 0)
+    (effects (font (size 2 2)) (justify left bottom))
+  )
+  (hierarchical_label "GND" (shape passive) (at 81.28 87.63 0)
     (effects (font (size 1.27 1.27)) (justify left))
   )
-  (hierarchical_label "RX" (shape input) (at 146.05 87.63 0)
+  (hierarchical_label "RX" (shape input) (at 125.73 43.18 0)
     (effects (font (size 1.27 1.27)) (justify left))
   )
-  (hierarchical_label "Vcc" (shape passive) (at 146.05 85.09 0)
+  (hierarchical_label "Vcc" (shape passive) (at 125.73 40.64 0)
     (effects (font (size 1.27 1.27)) (justify left))
   )
-  (hierarchical_label "SCK" (shape passive) (at 100.33 88.9 0)
+  (hierarchical_label "SCK" (shape passive) (at 81.28 45.72 0)
     (effects (font (size 1.27 1.27)) (justify left))
   )
-  (hierarchical_label "D8" (shape bidirectional) (at 124.46 97.79 0)
+  (hierarchical_label "D8" (shape bidirectional) (at 81.28 85.09 0)
     (effects (font (size 1.27 1.27)) (justify left))
   )
-  (hierarchical_label "SCK" (shape passive) (at 162.56 86.36 180)
+  (hierarchical_label "SCK" (shape passive) (at 115.57 73.66 180)
     (effects (font (size 1.27 1.27)) (justify right))
   )
-  (hierarchical_label "D7" (shape bidirectional) (at 124.46 95.25 0)
+  (hierarchical_label "D7" (shape bidirectional) (at 81.28 82.55 0)
     (effects (font (size 1.27 1.27)) (justify left))
   )
-  (hierarchical_label "GND" (shape passive) (at 146.05 82.55 0)
+  (hierarchical_label "GND" (shape passive) (at 125.73 38.1 0)
     (effects (font (size 1.27 1.27)) (justify left))
   )
-  (hierarchical_label "GND" (shape passive) (at 175.26 88.9 0)
+  (hierarchical_label "GND" (shape passive) (at 128.27 76.2 0)
     (effects (font (size 1.27 1.27)) (justify left))
   )
-  (hierarchical_label "D4" (shape bidirectional) (at 124.46 87.63 0)
+  (hierarchical_label "D4" (shape bidirectional) (at 81.28 74.93 0)
     (effects (font (size 1.27 1.27)) (justify left))
   )
-  (hierarchical_label "D6" (shape bidirectional) (at 124.46 92.71 0)
+  (hierarchical_label "D6" (shape bidirectional) (at 81.28 80.01 0)
     (effects (font (size 1.27 1.27)) (justify left))
   )
-  (hierarchical_label "RESET" (shape passive) (at 162.56 88.9 180)
+  (hierarchical_label "RESET" (shape passive) (at 115.57 76.2 180)
     (effects (font (size 1.27 1.27)) (justify right))
   )
-  (hierarchical_label "D3" (shape bidirectional) (at 124.46 85.09 0)
+  (hierarchical_label "D3" (shape bidirectional) (at 81.28 72.39 0)
     (effects (font (size 1.27 1.27)) (justify left))
   )
-  (hierarchical_label "MOSI" (shape input) (at 175.26 86.36 0)
+  (hierarchical_label "MOSI" (shape input) (at 128.27 73.66 0)
     (effects (font (size 1.27 1.27)) (justify left))
   )
-  (hierarchical_label "Vcc" (shape passive) (at 124.46 102.87 0)
+  (hierarchical_label "Vcc" (shape passive) (at 81.28 90.17 0)
     (effects (font (size 1.27 1.27)) (justify left))
   )
-  (hierarchical_label "D2" (shape bidirectional) (at 124.46 82.55 0)
+  (hierarchical_label "D2" (shape bidirectional) (at 81.28 69.85 0)
     (effects (font (size 1.27 1.27)) (justify left))
   )
-  (hierarchical_label "Vcc" (shape passive) (at 100.33 83.82 0)
+  (hierarchical_label "Vcc" (shape passive) (at 81.28 40.64 0)
     (effects (font (size 1.27 1.27)) (justify left))
   )
-  (hierarchical_label "D5" (shape bidirectional) (at 124.46 90.17 0)
+  (hierarchical_label "D5" (shape bidirectional) (at 81.28 77.47 0)
     (effects (font (size 1.27 1.27)) (justify left))
   )
-  (hierarchical_label "MISO" (shape output) (at 162.56 83.82 180)
+  (hierarchical_label "MISO" (shape output) (at 115.57 71.12 180)
     (effects (font (size 1.27 1.27)) (justify right))
   )
-  (hierarchical_label "GND" (shape passive) (at 100.33 81.28 0)
+  (hierarchical_label "GND" (shape passive) (at 81.28 38.1 0)
     (effects (font (size 1.27 1.27)) (justify left))
   )
-  (hierarchical_label "SDA" (shape bidirectional) (at 100.33 86.36 0)
+  (hierarchical_label "SDA" (shape bidirectional) (at 81.28 43.18 0)
     (effects (font (size 1.27 1.27)) (justify left))
   )
-  (hierarchical_label "TX" (shape output) (at 146.05 90.17 0)
+  (hierarchical_label "TX" (shape output) (at 125.73 45.72 0)
     (effects (font (size 1.27 1.27)) (justify left))
   )
-  (hierarchical_label "Vcc" (shape passive) (at 175.26 83.82 0)
+  (hierarchical_label "Vcc" (shape passive) (at 128.27 71.12 0)
     (effects (font (size 1.27 1.27)) (justify left))
   )
-  (symbol (lib_id "Connector_Generic:Conn_02x03_Odd_Even") (at 167.64 86.36 0) (unit 1)
+  (symbol (lib_id "Connector_Generic:Conn_02x03_Odd_Even") (at 120.65 73.66 0) (unit 1)
     (in_bom yes) (on_board yes)
-    (property "Reference" "J4" (id 0) (at 168.91 77.47 0))
-    (property "Value" "Conn_02x03_Odd_Even" (id 1) (at 168.91 80.01 0))
-    (property "Footprint" "Connector_PinHeader_2.54mm:PinHeader_1x09_P2.54mm_Vertical" (id 2) (at 167.64 86.36 0)
+    (property "Reference" "J4" (id 0) (at 121.92 64.77 0))
+    (property "Value" "Conn_02x03_Odd_Even" (id 1) (at 121.92 67.31 0))
+    (property "Footprint" "Connector_PinHeader_2.54mm:PinHeader_1x09_P2.54mm_Vertical" (id 2) (at 120.65 73.66 0)
       (effects (font (size 1.27 1.27)) hide)
     )
-    (property "Datasheet" "~" (id 3) (at 167.64 86.36 0)
+    (property "Datasheet" "~" (id 3) (at 120.65 73.66 0)
       (effects (font (size 1.27 1.27)) hide)
     )
@@
     (pin "6")
   )
-  (symbol (lib_id "Connector:Conn_01x04_Male") (at 95.25 83.82 0) (unit 1)
+  (symbol (lib_id "Connector:Conn_01x04_Male") (at 76.2 40.64 0) (unit 1)
     (in_bom yes) (on_board yes) (fields_autoplaced)
-    (property "Reference" "J1" (id 0) (at 95.885 76.2 0))
-    (property "Value" "Conn_01x04_Male" (id 1) (at 95.885 78.74 0))
-    (property "Footprint" "Connector_PinHeader_2.54mm:PinHeader_1x04_P2.54mm_Vertical" (id 2) (at 95.25 83.82 0)
+    (property "Reference" "J1" (id 0) (at 76.835 33.02 0))
+    (property "Value" "Conn_01x04_Male" (id 1) (at 76.835 35.56 0))
+    (property "Footprint" "Connector_PinHeader_2.54mm:PinHeader_1x04_P2.54mm_Vertical" (id 2) (at 76.2 40.64 0)
       (effects (font (size 1.27 1.27)) hide)
     )
-    (property "Datasheet" "~" (id 3) (at 95.25 83.82 0)
+    (property "Datasheet" "~" (id 3) (at 76.2 40.64 0)
       (effects (font (size 1.27 1.27)) hide)
     )
@@
     (pin "4")
   )
-  (symbol (lib_id "Connector:Conn_01x04_Male") (at 140.97 85.09 0) (unit 1)
+  (symbol (lib_id "Connector:Conn_01x04_Male") (at 120.65 40.64 0) (unit 1)
     (in_bom yes) (on_board yes) (fields_autoplaced)
-    (property "Reference" "J3" (id 0) (at 141.605 77.47 0))
-    (property "Value" "Conn_01x04_Male" (id 1) (at 141.605 80.01 0))
-    (property "Footprint" "Connector_PinHeader_2.54mm:PinHeader_1x04_P2.54mm_Vertical" (id 2) (at 140.97 85.09 0)
+    (property "Reference" "J3" (id 0) (at 121.285 33.02 0))
+    (property "Value" "Conn_01x04_Male" (id 1) (at 121.285 35.56 0))
+    (property "Footprint" "Connector_PinHeader_2.54mm:PinHeader_1x04_P2.54mm_Vertical" (id 2) (at 120.65 40.64 0)
       (effects (font (size 1.27 1.27)) hide)
     )
-    (property "Datasheet" "~" (id 3) (at 140.97 85.09 0)
+    (property "Datasheet" "~" (id 3) (at 120.65 40.64 0)
       (effects (font (size 1.27 1.27)) hide)
     )
@@
     (pin "4")
   )
-  (symbol (lib_id "Connector:Conn_01x09_Male") (at 119.38 92.71 0) (unit 1)
+  (symbol (lib_id "Connector:Conn_01x09_Male") (at 76.2 80.01 0) (unit 1)
     (in_bom yes) (on_board yes) (fields_autoplaced)
-    (property "Reference" "J2" (id 0) (at 120.015 77.47 0))
-    (property "Value" "Conn_01x09_Male" (id 1) (at 120.015 80.01 0))
-    (property "Footprint" "Connector_PinHeader_2.54mm:PinHeader_1x09_P2.54mm_Vertical" (id 2) (at 119.38 92.71 0)
+    (property "Reference" "J2" (id 0) (at 76.835 64.77 0))
+    (property "Value" "Conn_01x09_Male" (id 1) (at 76.835 67.31 0))
+    (property "Footprint" "Connector_PinHeader_2.54mm:PinHeader_1x09_P2.54mm_Vertical" (id 2) (at 76.2 80.01 0)
       (effects (font (size 1.27 1.27)) hide)
     )
-    (property "Datasheet" "~" (id 3) (at 119.38 92.71 0)
+    (property "Datasheet" "~" (id 3) (at 76.2 80.01 0)
       (effects (font (size 1.27 1.27)) hide)
     )

Commit message: Various refinements
Parts:
- J2: purpose (none) -> GPIO
- J4: purpose (none) -> ICSP
Changed lines of the file:
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@@
+      (effects (font (size 1.27 1.27)) hide)
+    )
+    (property "purpose" "ICSP" (id 4) (at 120.65 73.66 0)
       (effects (font (size 1.27 1.27)) hide)
     )
@@
       (effects (font (size 1.27 1.27)) hide)
     )
+    (property "purpose" "GPIO" (id 4) (at 76.2 80.01 0)
+      (effects (font (size 1.27 1.27)) hide)
+    )

Commit message: Verification
Parts:
- J4: footprint Connector_PinHeader_2.54mm:PinHeader_1x09_P2.54mm_Vertical -> Connector_PinHeader_2.54mm:PinHeader_2x03_P2.54mm_Vertical
Changed lines of the file:
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@@
     (property "Reference" "J4" (id 0) (at 121.92 64.77 0))
     (property "Value" "Conn_02x03_Odd_Even" (id 1) (at 121.92 67.31 0))
-    (property "Footprint" "Connector_PinHeader_2.54mm:PinHeader_1x09_P2.54mm_Vertical" (id 2) (at 120.65 73.66 0)
+    (property "Footprint" "Connector_PinHeader_2.54mm:PinHeader_2x03_P2.54mm_Vertical" (id 2) (at 120.65 73.66 0)
       (effects (font (size 1.27 1.27)) hide)
     )
