File: My MCU datalogger.kicad_pcb (KiCad board)
At the start: 4 copper layers, 47.7 x 30.6 mm, 31 parts, among them J1 Conn_01x04_Male, J2 Conn_01x09_Male, J3 Conn_01x04_Male, J4 Conn_02x03_Odd_Even, U1 24LC1025, U2 DS1307Z, U3 24LC1025, U4 ATMEGA328P-AU, Y1 32.768 KHz, Y2 16 MHz

Commit message: Final version
Routing:
- net Net-(C2-Pad2): track 44.4 -> 26.2 mm, vias 0 -> 2
- net Net-(C4-Pad2): track 18.3 -> 16.2 mm
- net /SDA: track 60.8 -> 59.5 mm
- net /D4: track 19.9 -> 20.5 mm
- net Net-(C3-Pad2): track 25.3 -> 24.7 mm
Other:
- board text added: "4"
- board text added: "4.6900 mm"
- board text added: "47.7044 mm x 30.6183 mm"
- board text removed: "1.6000 mm"
- board text removed: "2"
- board text removed: "47.7044 mm x 30.6182 mm"
